File: board/board.kicad_pcb (KiCad board)
At the start: 2 copper layers, 21 x 13 mm, 1 part

Commit message: initial
Parts:
- added J1: 009_1000BASE-T, on_edge:on_edge_2x05_device, F.Cu at (140.0, 96.5)
- added J2: Conn_01x08_Socket, b154:m12_x-code, F.Cu at (154.3, 96.7)
- moved LOGO1 2.44 mm to (147.8, 100.0)
Routing:
- net /m12-x-code/TD3+: track 0.00 -> 29.7 mm
- net /m12-x-code/TD3-: track 0.00 -> 27.0 mm
- net /m12-x-code/TD4+: track 0.00 -> 24.4 mm
- net /m12-x-code/TD4-: track 0.00 -> 19.5 mm
- net /m12-x-code/TD2-: track 0.00 -> 11.2 mm
- net /m12-x-code/TD1+: track 0.00 -> 10.8 mm
- net /m12-x-code/TD1-: track 0.00 -> 10.3 mm
- net /m12-x-code/TD2+: track 0.00 -> 9.72 mm
- net Earth: track 0.00 -> 4.79 mm, vias 0 -> 1
Other:
- outline, holes or cut-outs redrawn
- board text added: "osf.009"
- board text added: "osf.b154.v1.0"
